File: hardware/kicad/carrier_rev_a/carrier_rev_a.kicad_pcb (KiCad board)
At the start: 4 copper layers, 68 x 68 mm, 25 parts, among them J1 NHD-FFC40-0.5mm, J2 BMI088_HDR, J3 USB_C_Receptacle_HRO_TYPE-C-3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, J4 ENCODER_HDR, J5 TPS61169_HDR, J6 J6_SW_HDR, J7 J7_SW_HDR, U1 ESP32-S3-WROOM-1-N16R2, U2 TPS62162Q1_WSON8, U3 MCP23008-E_SO

Commit message: Generate carrier PCB Revision A validation reports
Connections:
- U1 pad 10: LCD_D13 -> LCD_D2
- U1 pad 11: LCD_D14 -> LCD_D1
- U1 pad 12: LCD_D4 -> LCD_D0
- U1 pad 17: LCD_D5 -> LCD_D9
- U1 pad 18: LCD_D6 -> LCD_D10
- U1 pad 19: LCD_D7 -> LCD_D11
- U1 pad 20: LCD_D8 -> LCD_D12
- U1 pad 21: LCD_D9 -> LCD_D13
- U1 pad 22: LCD_D10 -> LCD_D14
- U1 pad 24: IOX_SDA -> LCD_PCLK
- U1 pad 25: IOX_SCL -> LCD_DE
- U1 pad 31: LCD_HS -> (no net)
- U1 pad 32: LCD_VS -> BL_PWM
- U1 pad 35: BL_PWM -> IOX_INT
- U1 pad 36: SPARE -> IOX_SCL
- U1 pad 37: IOX_INT -> IOX_SDA
- U1 pad 38: LCD_DE -> LCD_VS
- U1 pad 39: LCD_PCLK -> LCD_HS
- U1 pad 4: LCD_D0 -> LCD_D8
- U1 pad 5: LCD_D1 -> LCD_D7
- U1 pad 6: LCD_D2 -> LCD_D6
- U1 pad 7: LCD_D3 -> LCD_D5
- U1 pad 8: LCD_D11 -> LCD_D4
- U1 pad 9: LCD_D12 -> LCD_D3
Routing:
- net GND: track 970.6 -> 925.5 mm
- net LCD_PCLK: track 56.5 -> 24.7 mm
- net LCD_DE: track 54.7 -> 25.5 mm
- net LCD_D14: track 46.6 -> 19.8 mm
- net LCD_D13: track 47.3 -> 20.6 mm
- net LCD_D11: track 48.9 -> 22.2 mm
- net LCD_D12: track 48.1 -> 21.4 mm
- net LCD_D0: track 48.0 -> 26.8 mm
- net LCD_D1: track 47.2 -> 28.6 mm
- net LCD_D2: track 46.4 -> 30.3 mm
- net LCD_D3: track 45.6 -> 32.1 mm
- net +3V3: track 295.6 -> 282.3 mm
- net LCD_D8: track 29.9 -> 41.0 mm
- net SPI_SCLK: track 69.9 -> 58.9 mm
- net SPI_MOSI: track 67.7 -> 56.7 mm
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