File: hardware/kicad/carrier_rev_a/carrier_rev_a.kicad_sch (KiCad schematic)
At the start: 19 parts, among them J1 NHD-2.1-480480AF-ASXP FFC, J2 BMI088 Shuttle, J3 USB-C 2.0, J4 Bourns PEC09, J5 TPS61169 Interface, U1 ESP32-S3-WROOM-1-N16R2, U2 TPS62162-Q1, U3 MCP23008-E/SO

Commit message: Generate carrier PCB Revision A validation reports
Connections:
- net SPARE is gone; now on net IOX_SCL: U1.27 (IO0)
- net BL_PWM: now also U1.31 (IO38); no longer U1.28 (IO35)
- net IOX_INT: now also U1.28 (IO35); no longer U1.26 (IO45)
- net IOX_SCL: no longer U1.38 (IO2)
- net IOX_SDA: now also U1.26 (IO45); no longer U1.39 (IO1)
- net LCD_D0: now also U1.10 (IO17); no longer U1.18 (IO10)
- net LCD_D1: now also U1.11 (IO18); no longer U1.17 (IO9)
- net LCD_D10: now also U1.4 (IO4); no longer U1.41 (EPAD_GND)
- net LCD_D11: now also U1.3 (EN); no longer U1.14 (IO20_USB_D+)
- net LCD_D12: now also U1.2 (3V3); no longer U1.13 (IO19_USB_D-)
- net LCD_D13: now also U1.1 (GND); no longer U1.12 (IO8)
- net LCD_D14: now also U1.41 (EPAD_GND); no longer U1.11 (IO18)
- net LCD_D2: now also U1.12 (IO8); no longer U1.16 (IO46)
- net LCD_D3: now also U1.13 (IO19_USB_D-); no longer U1.15 (IO3)
- net LCD_D4: now also U1.14 (IO20_USB_D+); no longer U1.10 (IO17)
- net LCD_D5: now also U1.15 (IO3); no longer U1.5 (IO5)
- net LCD_D6: now also U1.16 (IO46); no longer U1.4 (IO4)
- net LCD_D7: now also U1.17 (IO9); no longer U1.3 (EN)
- net LCD_D8: now also U1.18 (IO10); no longer U1.2 (3V3)
- net LCD_D9: now also U1.5 (IO5); no longer U1.1 (GND)
- net LCD_DE: now also U1.38 (IO2); no longer U1.25 (IO48)
- net LCD_HS: now also U1.24 (IO47); no longer U1.32 (IO39)
- net LCD_PCLK: now also U1.39 (IO1); no longer U1.24 (IO47)
- net LCD_VS: now also U1.25 (IO48); no longer U1.31 (IO38)
- no-connect marks 13 -> 14
